File: KiCad/ColorTimer-ESP12F.kicad_sch (KiCad schematic)
At the start: 40 parts, among them J1 SW_CON, J2 USB_B_Micro, J3 COLOER_LED, J4 AkitsukiCON, J5 GPIO_CON, J6 POWER_CON, Q1 2N7000, Q2 2N7000, SW1 RESET, SW2 Trigger SW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

Commit message: 微修正、ガーバー再出力
Parts:
- R10: value 330 -> 1k
Changed lines of the file:
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@@
 			)
 		)
-		(property "Value" "330"
+		(property "Value" "1k"
 			(at 203.2 134.6199 0)
 			(effects

Commit message: 表面実装部品版 作成開始
Parts:
- removed C3: 10u, Capacitor_THT:C_Disc_D3.0mm_W1.6mm_P2.50mm, symbol Device:C_Small
- removed C4: 1u, Capacitor_THT:C_Disc_D3.0mm_W1.6mm_P2.50mm, symbol Device:C_Small
- removed C7: 22u, Capacitor_THT:CP_Radial_D5.0mm_P2.50mm, symbol Device:C_Polarized
- removed J2: USB_B_Micro, Connector_USB:USB_Micro-B_Molex-105017-0001, symbol Connector:USB_B_Micro
- removed J4: AkitsukiCON, AE:AE-USB-MICRO-B-D, symbol Connector_Generic:Conn_01x05
- removed J5: GPIO_CON, Connector_PinSocket_2.54mm:PinSocket_1x09_P2.54mm_Vertical, symbol Connector_Generic:Conn_01x09
- removed Q1, Q2: 2N7000, Package_TO_SOT_THT:TO-92_Inline_Wide, symbol Transistor_FET:2N7000
- removed R6: 33, Resistor_THT:R_Axial_DIN0207_L6.3mm_D2.5mm_P10.16mm_Horizontal, symbol Device:R_Small_US
- removed SW3: FLASH, Button_Switch_THT:SW_PUSH_6mm_H8mm, symbol Switch:SW_Push
- removed U2: CH340K, Package_SO:SSOP-10-1EP_3.9x4.9mm_P1mm_EP2.1x3.3mm, symbol Interface_USB:CH340K
- removed U3: BA033CC0T_TO220, Package_TO_SOT_THT:TO-220-3_Vertical, symbol Regulator_Linear:LM7805_TO220
- added D4: D_Schottky, Diode_SMD:D_SOD-123, symbol Device:D_Schottky
- added J2: OLED, Connector_JST:JST_XH_B4B-XH-A_1x04_P2.50mm_Vertical, symbol Connector_Generic:Conn_01x04
- added J4: Ext_Con, Connector_JST:JST_XH_B3B-XH-A_1x03_P2.50mm_Vertical, symbol Connector_Generic:Conn_01x03
- added J5: Downloader_CON, Connector_PinSocket_2.54mm:PinSocket_1x06_P2.54mm_Vertical, symbol Connector_Generic:Conn_01x06
- added J7: POWER_CON, Connector_JST:JST_XH_B2B-XH-A_1x02_P2.50mm_Vertical, symbol Connector_Generic:Conn_01x02
- added U2: AMS1117-3.3, Package_TO_SOT_SMD:SOT-223-3_TabPin2, symbol Regulator_Linear:AMS1117-3.3
- C1, C2: footprint Capacitor_THT:C_Disc_D3.0mm_W1.6mm_P2.50mm -> Capacitor_SMD:C_0603_1608Metric_Pad1.08x0.95mm_HandSolder
- C5, C6: value 0.1u -> 22u; footprint Capacitor_THT:C_Disc_D3.0mm_W1.6mm_P2.50mm -> Capacitor_SMD:C_0603_1608Metric_Pad1.08x0.95mm_HandSolder
- D1, D2, D3: footprint LED_THT:LED_D3.0mm -> LED_SMD:LED_0603_1608Metric_Pad1.05x0.95mm_HandSolder
- J1: footprint Connector_PinSocket_2.54mm:PinSocket_1x02_P2.54mm_Vertical -> Connector_JST:JST_XH_B2B-XH-A_1x02_P2.50mm_Vertical
- J3: footprint Connector_PinSocket_2.54mm:PinSocket_1x03_P2.54mm_Vertical -> Connector_JST:JST_XH_B3B-XH-A_1x03_P2.50mm_Vertical
- J6: value POWER_CON -> POWER_SW_CON; footprint Connector_PinSocket_2.54mm:PinSocket_1x02_P2.54mm_Vertical -> Connector_JST:JST_XH_B2B-XH-A_1x02_P2.50mm_Vertical
- R1, R10, R2, R3, R7, R8, R9: footprint Resistor_THT:R_Axial_DIN0207_L6.3mm_D2.5mm_P10.16mm_Horizontal -> Resistor_SMD:R_0603_1608Metric_Pad0.98x0.95mm_HandSolder
- R4, R5: value 330 -> 1k; footprint Resistor_THT:R_Axial_DIN0207_L6.3mm_D2.5mm_P10.16mm_Horizontal -> Resistor_SMD:R_0603_1608Metric_Pad0.98x0.95mm_HandSolder
- SW1, SW2: footprint Button_Switch_THT:SW_PUSH_6mm_H8mm -> Button_Switch_SMD:SW_Push_SPST_NO_Alps_SKRK
Connections:
- net +3.3V: now also C6.1, D4.1 (K), J2.3 (Pin_3), J5.1 (Pin_1)
- net +5V: now also R10.2, U2.3 (VI)
- net ADC: now also J4.2 (Pin_2)
- net EN: now also J5.4 (Pin_4); no longer C6.1
- net GND: now also J3.2 (Pin_2), J2.4 (Pin_4), J4.3 (Pin_3), J5.6 (Pin_6), J7.2 (Pin_2), U2.1 (GND)
- net GPIO0: now also J5.5 (Pin_5)
- net GPIO14: now also J4.1 (Pin_1)
- net GPIO4: now also J2.1 (Pin_1)
- net GPIO5: now also J2.2 (Pin_2)
- net RxD: now also J5.3 (Pin_3)
- net TxD: now also J5.2 (Pin_2)
- net VCC: no longer R10.2
- net at F1.1: now also J7.1 (Pin_1)
- net GPIO12: no longer names the net of J3.3 (Pin_3), R5.2, U1.6 (GPIO12)
- net GPIO13: no longer names the net of J3.1 (Pin_1), R4.2, U1.7 (GPIO13)
- net GPIO16: no longer names the net of J1.1 (Pin_1), R2.2, SW2.2, U1.4 (GPIO16)
- new net: D4.2 (A), U2.2 (VO)
- no-connect marks 10 -> 7
Other:
- note added: "+3.3V"
- note added: "EN"
- note added: "GPIO0"
- note added: "RxD"
- note added: "TxD"
- note removed: "D+"
- note removed: "D-"
- note removed: "NC"
- note removed: "VBAS"
- moved on the sheet: D3, J6, R10

Commit message: REV2 表面実装部品版 ガーバーデータ出力
Parts:
- removed J4: Ext_Con, Connector_JST:JST_XH_B3B-XH-A_1x03_P2.50mm_Vertical, symbol Connector_Generic:Conn_01x03
- added J4: ADC_CON, Connector_JST:JST_XH_B2B-XH-A_1x02_P2.50mm_Vertical, symbol Connector_Generic:Conn_01x02
- added J8: IO14_CON, Connector_JST:JST_XH_B2B-XH-A_1x02_P2.50mm_Vertical, symbol Connector_Generic:Conn_01x02
- added R11, R12: 2.4k, Resistor_SMD:R_0603_1608Metric_Pad0.98x0.95mm_HandSolder, symbol Device:R_Small_US
Connections:
- net +3.3V: now also R11.1, R12.1; no longer C6.1
- net ADC: now also J4.1 (Pin_1)
- net GND: now also J4.2 (Pin_2), J8.2 (Pin_2)
- net GPIO14: now also J8.1 (Pin_1)
- net GPIO4: now also R11.2
- net GPIO5: now also R12.2
- net at D4.2 (A), U2.2 (VO): now also C6.1
Other:
- moved on the sheet: C6, D4, J2

Commit message: REV2 2色LEDのGNDに33Ω追加、ガーバー再出力 試作用
Parts:
- added R6: 33, Resistor_SMD:R_0603_1608Metric_Pad0.98x0.95mm_HandSolder, symbol Device:R_Small_US
Connections:
- net GND: now also R6.1; no longer J3.2 (Pin_2)
- new net: J3.2 (Pin_2), R6.2
Changed lines of the file:
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@@
 	(wire
 		(pts
+			(xy 105.41 133.35) (xy 105.41 138.43)
+		)
+		(stroke
+			(width 0)
+			(type default)
+		)
+	)
+	(wire
+		(pts
 			(xy 160.02 54.61) (xy 160.02 83.82)
 		)
@@
 	(wire
 		(pts
-			(xy 105.41 119.38) (xy 105.41 130.81)
+			(xy 105.41 119.38) (xy 105.41 128.27)
 		)
 		(stroke
@@
 	)
 	(symbol
+		(lib_id "Device:R_Small_US")
+		(at 105.41 130.81 180)
+		(unit 1)
+		(exclude_from_sim no)
+		(in_bom yes)
+		(on_board yes)
+		(dnp no)
+		(fields_autoplaced yes)
+		(property "Reference" "R6"
+			(at 107.95 129.5399 0)
+			(effects
+				(font
+					(size 1.27 1.27)
+				)
+				(justify right)
+			)
+		)
+		(property "Value" "33"
+			(at 107.95 132.0799 0)
+			(effects
+				(font
+					(size 1.27 1.27)
+				)
+				(justify right)
+			)
+		)
+		(property "Footprint" "Resistor_SMD:R_0603_1608Metric_Pad0.98x0.95mm_HandSolder"
+			(at 105.41 130.81 0)
+			(effects
+				(font
+					(size 1.27 1.27)
+				)
+				(hide yes)
+			)
+		)
+		(property "Datasheet" "~"
+			(at 105.41 130.81 0)
+			(effects
+				(font
+					(size 1.27 1.27)
+				)
+				(hide yes)
+			)
+		)
+		(property "Description" "Resistor, small US symbol"
+			(at 105.41 130.81 0)
+			(effects
+				(font
+					(size 1.27 1.27)
+				)
+				(hide yes)
+			)
+		)
+		(pin "1"
+		)
+		(pin "2"
+		)
+		(instances
+			(project "ColorTimer-ESP12F"
+				(path "/3ff58839-42d9-41e5-8791-30721827b8bc"
+					(reference "R6")
+					(unit 1)
+				)
+			)
+		)
+	)
+	(symbol
 		(lib_id "ESP8266Lib:ESP-12F")
 		(at 116.84 54.61 0)
@@
 	(symbol
 		(lib_id "power:GND")
-		(at 105.41 130.81 0)
+		(at 105.41 138.43 0)
 		(unit 1)
 		(exclude_from_sim no)
@@
 		(fields_autoplaced yes)
 		(property "Reference" "#PWR010"
-			(at 105.41 137.16 0)
+			(at 105.41 144.78 0)
 			(effects
 				(font
@@
 		)
 		(property "Value" "GND"
-			(at 105.41 135.89 0)
+			(at 105.41 143.51 0)
 			(effects
 				(font
@@
 		)
 		(property "Footprint" ""
-			(at 105.41 130.81 0)
+			(at 105.41 138.43 0)
 			(effects
 				(font
@@
 		)
 		(property "Datasheet" ""
-			(at 105.41 130.81 0)
+			(at 105.41 138.43 0)
 			(effects
 				(font
@@
 		)
 		(property "Description" "Power symbol creates a global label with name \"GND\" , ground"
-			(at 105.41 130.81 0)
+			(at 105.41 138.43 0)
 			(effects
 				(font
