File: KiCad/ColorTimer-ESP12F.kicad_sch (KiCad schematic)
At the start: 40 parts, among them J1 SW_CON, J2 USB_B_Micro, J3 COLOER_LED, J4 AkitsukiCON, J5 GPIO_CON, J6 POWER_CON, Q1 2N7000, Q2 2N7000, SW1 RESET, SW2 Trigger SW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

Commit message: REV1.1 回路検討
Parts:
- removed C7: 22u, Capacitor_THT:CP_Radial_D5.0mm_P2.50mm, symbol Device:C_Polarized
- removed J5: GPIO_CON, Connector_PinSocket_2.54mm:PinSocket_1x09_P2.54mm_Vertical, symbol Connector_Generic:Conn_01x09
- removed J6: POWER_CON, Connector_PinSocket_2.54mm:PinSocket_1x02_P2.54mm_Vertical, symbol Connector_Generic:Conn_01x02
- removed R1, R2, R3, R7, R9: 10k, Resistor_THT:R_Axial_DIN0207_L6.3mm_D2.5mm_P10.16mm_Horizontal, symbol Device:R_Small_US
- removed U3: BA033CC0T_TO220, Package_TO_SOT_THT:TO-220-3_Vertical, symbol Regulator_Linear:LM7805_TO220
- added C7: 22u, Capacitor_THT:C_Disc_D3.0mm_W1.6mm_P2.50mm, symbol Device:C_Small
- added D4: D_Schottky, symbol Device:D_Schottky
- added J10: ADC_CON, Connector_PinSocket_2.54mm:PinSocket_1x02_P2.54mm_Vertical, symbol Connector_Generic:Conn_01x02
- added J11: POWER_CON_5V, Connector_PinSocket_2.54mm:PinSocket_1x02_P2.54mm_Vertical, symbol Connector_Generic:Conn_01x02
- added J5: OLED_CON, symbol Connector_Generic:Conn_01x04
- added J6: USB_SERIAL, symbol Connector_Generic:Conn_01x06
- added J7: POWER_SW, Connector_PinSocket_2.54mm:PinSocket_1x02_P2.54mm_Vertical, symbol Connector_Generic:Conn_01x02
- added J8: TORIGGER_SW, Connector_PinSocket_2.54mm:PinSocket_1x02_P2.54mm_Vertical, symbol Connector_Generic:Conn_01x02
- added J9: IO14_CON, Connector_PinSocket_2.54mm:PinSocket_1x02_P2.54mm_Vertical, symbol Connector_Generic:Conn_01x02
- added R11, R12: 2.4k, Resistor_THT:R_Axial_DIN0207_L6.3mm_D2.5mm_P10.16mm_Horizontal, symbol Device:R_Small_US
- added RN1: 10k, Resistor_THT:R_Array_SIP9, symbol Device:R_Network08_US
- added U3: AMS1117-3.3, Package_TO_SOT_SMD:SOT-223-3_TabPin2, symbol Regulator_Linear:AMS1117-3.3
- C5: value 0.1u -> 22u
- J1: value SW_CON -> POWER_CON_3.3V
Connections:
- net +3.3V: now also J1.1 (Pin_1), R10.2, C7.1, D4.1 (K), J5.3 (Pin_3), R11.1, R12.1, RN1.1 (common)
- net +5V: now also J7.2 (Pin_2), U3.3 (VI)
- net ADC: now also J10.1 (Pin_1)
- net DTR: now also J6.6 (Pin_6)
- net EN: now also RN1.4 (R3)
- net GND: now also C7.2, J10.2 (Pin_2), J11.2 (Pin_2), J5.4 (Pin_4), J6.1 (Pin_1), J8.2 (Pin_2), J9.2 (Pin_2), U3.1 (GND)
- net GPIO0: now also RN1.5 (R4)
- net GPIO14: now also J9.1 (Pin_1)
- net GPIO4: now also J5.1 (Pin_1), R11.2
- net GPIO5: now also J5.2 (Pin_2), R12.2
- net RTS: now also J6.2 (Pin_2)
- net RxD: now also J6.4 (Pin_4)
- net TxD: now also J6.5 (Pin_5)
- net VCC: now also J11.1 (Pin_1), J6.3 (Pin_3), J7.1 (Pin_1); no longer R10.2
- net RESET: now reaches C1.1, SW1.2, U1.1 (REST)
- net RESET: now also RN1.3 (R2)
- net at U1.11 (GPIO2): now also RN1.6 (R5)
- net GPIO12: no longer names the net of J3.3 (Pin_3), R5.2, U1.6 (GPIO12)
- net GPIO13: no longer names the net of J3.1 (Pin_1), R4.2, U1.7 (GPIO13)
- net GPIO16: no longer names the net of SW2.2, U1.4 (GPIO16)
- net GPIO16: now also J8.1 (Pin_1), RN1.2 (R1); no longer J1.1 (Pin_1)
- new net: D4.2 (A), U3.2 (VO)
- no-connect marks 10 -> 13
Other:
- note added: "+5V"
- note added: "DTR"
- note added: "RTS(CTS)"
- note added: "RxD"
- note added: "TxD"
- moved on the sheet: C5, C6, D3, J3, Q1, Q2, R10, R6, SW4
